File: kicad/PoE_PD_Interface.sch (KiCad schematic (older format))
At the start: 11 parts, among them U2 NCP1090, U3 PG02S4805A

Commit message: Add files via upload
Parts:
- R10: renamed from R8; footprint Resistor_SMD:R_0603_1608Metric -> Resistor_SMD:R_0805_2012Metric
- R8: renamed from R6; footprint Resistor_SMD:R_0603_1608Metric -> Resistor_SMD:R_0805_2012Metric
- R9: renamed from R7; footprint Resistor_SMD:R_0603_1608Metric -> Resistor_SMD:R_0805_2012Metric
- renumbered C11 to C10, C12 to C11, C13 to C12, D1 to D3, D2 to D4, D3 to D5
Other:
- note added: "802.3af Power over Ethernet"
- moved on the sheet: C10, C11, C12, D3, D4, D5, R10, R8, R9, U2, U3
