File: kicad/Relay_Interface.sch (KiCad schematic (older format))
At the start: 24 parts, among them J3 SJ1-2503A, J4 SJ1-2503A, J5 SJ1-2503A, K1 G5LE-14_DC3, K2 G5LE-14_DC3, K3 G5LE-14_DC3, Q1 BC846B_215, Q2 BC846B_215, Q3 BC846B_215, U5 LTV-817S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

Commit message: Add files via upload
Parts:
- D10: renamed from D6; value LED -> BLUE; footprint LED_SMD:LED_0805_2012Metric -> LED_SMD:LED_1206_3216Metric_Pad1.42x1.75mm_HandSolder
- D8: renamed from D4; value LED -> BLUE; footprint LED_SMD:LED_0805_2012Metric -> LED_SMD:LED_1206_3216Metric_Pad1.42x1.75mm_HandSolder
- D9: renamed from D5; value LED -> BLUE; footprint LED_SMD:LED_0805_2012Metric -> LED_SMD:LED_1206_3216Metric_Pad1.42x1.75mm_HandSolder
- R18: renamed from R13; value 1k -> 100; footprint Resistor_SMD:R_0603_1608Metric -> Resistor_SMD:R_0805_2012Metric
- R19: renamed from R14; value 1k -> 100; footprint Resistor_SMD:R_0603_1608Metric -> Resistor_SMD:R_0805_2012Metric
- R20: renamed from R15; value 1k -> 100; footprint Resistor_SMD:R_0603_1608Metric -> Resistor_SMD:R_0805_2012Metric
- R21: renamed from R16; value 510 -> 1k; footprint Resistor_SMD:R_0603_1608Metric -> Resistor_SMD:R_0805_2012Metric
- R22: renamed from R17; value 510 -> 1k; footprint Resistor_SMD:R_0603_1608Metric -> Resistor_SMD:R_0805_2012Metric
- R23: renamed from R18; value 510 -> 1k; footprint Resistor_SMD:R_0603_1608Metric -> Resistor_SMD:R_0805_2012Metric
- renumbered D7 to D11, D8 to D12, D9 to D13, J3 to J5, J4 to J6, J5 to J7
Other:
- note added: "Door 1 Relay"
- note added: "Door 2 Relay"
- note added: "Door 3 Relay"
- moved on the sheet: D10, D11, D12, D13, D8, D9, J5, J6, J7, K1, K2, K3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
