File: kicad/W5100_Ethernet_Interface.sch (KiCad schematic (older format))
At the start: 16 parts, among them U4 W5500, X2 SPI Disconnect, Y2 25MHz

Commit message: Add files via upload
Parts:
- removed R10: 10k, Resistor_SMD:R_0603_1608Metric, symbol Device:R
- added C13, C14: 10u/16V, Capacitor_SMD:C_0805_2012Metric, symbol Device:CP1
- added C15, C16: 100n, Capacitor_SMD:C_0805_2012Metric, symbol Device:C
- added D6: GREEN, LED_SMD:LED_1206_3216Metric_Pad1.42x1.75mm_HandSolder, symbol Device:LED
- added D7: YELLOW, LED_SMD:LED_1206_3216Metric_Pad1.42x1.75mm_HandSolder, symbol Device:LED
- added R12, R13: 10k, Resistor_SMD:R_0805_2012Metric, symbol Device:R
- added R16, R17: 330, Resistor_SMD:R_0805_2012Metric, symbol Device:R
- C17: renamed from C14; footprint Capacitor_SMD:C_0603_1608Metric -> Capacitor_SMD:C_0805_2012Metric
- C18: renamed from C15; footprint Capacitor_SMD:C_0603_1608Metric -> Capacitor_SMD:C_0805_2012Metric
- C19: renamed from C16; footprint Capacitor_SMD:C_0603_1608Metric -> Capacitor_SMD:C_0805_2012Metric
- C20: renamed from C17; footprint Capacitor_SMD:C_0603_1608Metric -> Capacitor_SMD:C_0805_2012Metric
- C21: renamed from C18; footprint Capacitor_SMD:C_0603_1608Metric -> Capacitor_SMD:C_0805_2012Metric
- C22: renamed from C19; footprint Capacitor_SMD:C_0603_1608Metric -> Capacitor_SMD:C_0805_2012Metric
- C23: renamed from C20; footprint Capacitor_SMD:C_0603_1608Metric -> Capacitor_SMD:C_0805_2012Metric
- R11: footprint Resistor_SMD:R_0603_1608Metric -> Resistor_SMD:R_0805_2012Metric
- R14: renamed from R9; footprint Resistor_SMD:R_0603_1608Metric -> Resistor_SMD:R_0805_2012Metric
- R15: renamed from R12; footprint Resistor_SMD:R_0603_1608Metric -> Resistor_SMD:R_0805_2012Metric
- U4: footprint digikey-footprints:LQFP-48_7x7mm -> Package_QFP:LQFP-48_7x7mm_P0.5mm
- Y2: footprint Crystal:Crystal_SMD_HC49-SD -> Crystal:Crystal_SMD_5032-2Pin_5.0x3.2mm
- renumbered C21 to C24, C22 to C25, X2 to X4
Connections:
- net +3V3: now also R11.1, C13.1, C14.1, C15.1, C16.1, D6.1 (K), D7.1 (K), R12.1, R13.1; no longer R11.2, U4.43 (PMODE2), U4.44 (PMODE1), U4.45 (PMODE0)
- net GND: now also C13.2, C14.2, C15.2, C16.2
- net W_INT: no longer R11.1
- net at U4.25 (LINKLED): now also R17.2
- net at U4.27 (ACTLED): now also R16.2
- new net: R13.2, U4.43 (PMODE2)
- new net: R12.2, U4.44 (PMODE1)
- new net: R11.2, U4.45 (PMODE0)
- new net: D6.2 (A), R16.1
- new net: D7.2 (A), R17.1
- no-connect marks 16 -> 14
Other:
- note added: "W5500 Ethernet Network Access"
- note added: "W5500 SPI Disconnect\nfor Programming"
- moved on the sheet: C17, C18, C19, C20, C21, C22, C23, C24, C25, R14, R15, U4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
