File: kicad/garHAge_v2.sch (KiCad schematic (older format))
At the start: 24 parts, among them J1 0813-1X1T-57-F, J2 Serial Interface, J6 SJ1-2503A, J7 SJ1-2503A, J8 SJ1-2503A, U1 ATMEGA328P-AU, X1 ICSP, Y1 8MHz

Commit message: Add files via upload
Parts:
- removed C4: 100n, Capacitor_SMD:C_0603_1608Metric, symbol Device:C
- added D1: BLUE, LED_SMD:LED_1206_3216Metric_Pad1.42x1.75mm_HandSolder, symbol Device:LED
- added D2: RED, LED_SMD:LED_1206_3216Metric_Pad1.42x1.75mm_HandSolder, symbol Device:LED
- added R5, R7: 330, Resistor_SMD:R_0805_2012Metric, symbol Device:R
- added X2: Serial Pwr Disconnect, Connector_PinHeader_2.54mm:PinHeader_1x02_P2.54mm_Vertical, symbol Connector_Generic:Conn_01x02
- C1, C2: value 10n -> 6.8n; footprint Capacitor_SMD:C_0603_1608Metric -> Capacitor_SMD:C_0805_2012Metric
- C3: value 100n -> 22n; footprint Capacitor_SMD:C_0603_1608Metric -> Capacitor_SMD:C_0805_2012Metric
- C4: renamed from C5; value 100n -> 10n; footprint Capacitor_SMD:C_0603_1608Metric -> Capacitor_SMD:C_0805_2012Metric
- C7: renamed from C6; footprint Capacitor_SMD:C_0603_1608Metric -> Capacitor_SMD:C_0805_2012Metric
- C8: renamed from C9; footprint Capacitor_SMD:C_0603_1608Metric -> Capacitor_SMD:C_0805_2012Metric
- C9: renamed from C10; footprint Capacitor_SMD:C_0603_1608Metric -> Capacitor_SMD:C_0805_2012Metric
- L1: footprint Capacitor_SMD:C_0603_1608Metric -> Capacitor_SMD:C_0805_2012Metric
- R6: renamed from R5; footprint Resistor_SMD:R_0603_1608Metric -> Resistor_SMD:R_0805_2012Metric
- Y1: footprint Crystal:Crystal_SMD_HC49-SD -> Crystal:Crystal_SMD_5032-2Pin_5.0x3.2mm
- renumbered C7 to C5, C8 to C6, J6 to J1, J7 to J2, J8 to J3, J1 to J4, J2 to X3
Connections:
- net labels added: BOOT_STATUS, CT, D1SENSOR, D2SENSOR, D3SENSOR, RD+, RD-
- wire segments 149 -> 155
- no-connect marks 15 -> 14
Other:
- note added: "ATMEGA328P MCU"
- note added: "Ethernet and 802.3af PoE\nInterface"
- note added: "ICSP Interface"
- note added: "Power Indication"
- note added: "Reed Switch Interface"
- note added: "Relay Interface"
- note added: "Serial Debug Interface"
- moved on the sheet: C1, C2, C3, C4, C5, C6, C7, C8, C9, J1, J2, J3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
